File: Hardware/Gator_Air.brd (EAGLE design)
At the start: 38.1 x 25.4 mm, 59 parts, among them J1 GATORGATOR_MINI, J2 GATORGATOR_MINI, J3 GATORGATOR_MINI, J4 GATORGATOR_MINI, J5 GATORGATOR_MINI, J6 GATORGATOR_MINI, J7 GATORGATOR_MINI, J8 GATORGATOR_MINI, Q1 2.5A/30V/105mΩ, U2 CCS811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

Commit message: post checklist changes
Parts:
- moved LOGO4 2.54 mm to (19.1, 3.81)
Changed lines of the file:
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@@
 <attribute name="VALUE" x="2.54" y="10.668" size="0.6096" layer="27" font="vector" ratio="20" align="top-center"/>
 </element>
-<element name="LOGO4" library="SparkFun-Aesthetics" package="OSHW-LOGO-S" value="OSHW-LOGOS" x="19.05" y="1.27" smashed="yes" rot="MR0"/>
+<element name="LOGO4" library="SparkFun-Aesthetics" package="OSHW-LOGO-S" value="OSHW-LOGOS" x="19.05" y="3.81" smashed="yes" rot="MR0"/>
 <element name="FD1" library="SparkFun-Aesthetics" package="FIDUCIAL-1X2" value="FIDUCIAL1X2" x="36.83" y="16.51" smashed="yes"/>
 <element name="FD2" library="SparkFun-Aesthetics" package="FIDUCIAL-1X2" value="FIDUCIAL1X2" x="1.27" y="8.89" smashed="yes"/>
@@
 <wire x1="26.915" y1="13.645" x2="25.583" y2="13.645" width="0.2032" layer="1"/>
 <wire x1="25.583" y1="13.645" x2="25.4" y2="13.462" width="0.2032" layer="1"/>
-<wire x1="11.01" y1="17.78" x2="12.7" y2="17.78" width="0.2032" layer="1"/>
-<via x="12.7" y="17.78" extent="1-16" drill="0.381"/>
-<wire x1="12.7" y1="17.78" x2="11.176" y2="16.256" width="0.2032" layer="16"/>
-<wire x1="11.176" y1="16.256" x2="11.176" y2="11.303" width="0.2032" layer="16"/>
+<via x="12.7" y="16.51" extent="1-16" drill="0.381"/>
+<wire x1="12.7" y1="16.51" x2="11.176" y2="14.986" width="0.2032" layer="16"/>
+<wire x1="11.176" y1="14.986" x2="11.176" y2="11.303" width="0.2032" layer="16"/>
 <via x="11.176" y="11.303" extent="1-16" drill="0.381"/>
 <wire x1="25.4" y1="17.78" x2="22.606" y2="17.78" width="0.2032" layer="16"/>
@@
 <wire x1="17.78" y1="17.995" x2="17.78" y2="19.05" width="0.2032" layer="1"/>
 <wire x1="20.32" y1="17.995" x2="20.32" y2="19.05" width="0.2032" layer="1"/>
-<wire x1="15.24" y1="17.78" x2="16.51" y2="19.05" width="0.2032" layer="1"/>
+<wire x1="13.97" y1="16.51" x2="16.51" y2="19.05" width="0.2032" layer="1"/>
 <wire x1="16.51" y1="19.05" x2="17.78" y2="19.05" width="0.2032" layer="1"/>
-<wire x1="12.7" y1="17.78" x2="15.24" y2="17.78" width="0.2032" layer="1"/>
+<wire x1="12.7" y1="16.51" x2="13.97" y2="16.51" width="0.2032" layer="1"/>
 <contactref element="R1" pad="2"/>
 <contactref element="Q1" pad="2"/>
@@
 <wire x1="11.176" y1="11.303" x2="8.216" y2="11.303" width="0.1778" layer="1"/>
 <wire x1="8.216" y1="11.303" x2="7.239" y2="10.326" width="0.1778" layer="1"/>
+<wire x1="12.7" y1="16.51" x2="11.43" y2="16.51" width="0.1778" layer="1"/>
+<wire x1="11.43" y1="16.51" x2="11.01" y2="16.93" width="0.1778" layer="1"/>
+<wire x1="11.01" y1="16.93" x2="11.01" y2="17.78" width="0.1778" layer="1"/>
 </signal>
 <signal name="!RST">
