File: Hardware/Gator_Environment.brd (EAGLE design)
At the start: 38.1 x 25.4 mm, 59 parts, among them J1 GATORGATOR_MINI, J2 GATORGATOR_MINI, J3 GATORGATOR_MINI, J4 GATORGATOR_MINI, J5 GATORGATOR_MINI, J6 GATORGATOR_MINI, J7 GATORGATOR_MINI, J8 GATORGATOR_MINI, Q1 2.5A/30V/105mΩ, U2 CCS811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

Commit message: engineer run of checklist
Parts:
- removed U$17: (no value), buzzard_labels (4):GATOR#AIR0
- added U$25: (no value), buzzard_labels (12):GATOR#ENVIRONMENT0
- moved D4 1.91 mm to (19.1, 7.62)
- moved U$18 1.78 mm to (16.6, 9.53)
- moved U$14 0.13 mm to (36.4, 7.75)
- moved U$13 0.13 mm to (26.5, 7.75)
Routing:
- net SCL: track 51.9 -> 49.9 mm
- net N$2: track 1.92 -> 3.82 mm
- net SDA: track 44.5 -> 42.6 mm
Other:
- board text added: "v10"
- board text removed: "v01"
Changed lines of the file:
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@@
 <wire x1="38.1" y1="25.4" x2="38.1" y2="0" width="0.2032" layer="20"/>
 <wire x1="38.1" y1="0" x2="0" y2="0" width="0.2032" layer="20"/>
-<text x="19.05" y="0.92075" size="1.016" layer="16" font="vector" ratio="20" rot="MR180" align="center">v01</text>
+<text x="19.05" y="0.92075" size="1.016" layer="16" font="vector" ratio="20" rot="MR180" align="center">v10</text>
 <text x="8.509" y="10.414" size="0.6096" layer="25">CCS811</text>
 <text x="14.859" y="10.541" size="0.6096" layer="25">BME280</text>
-<text x="16.51" y="-21.59" size="1.778" layer="51">Andrew England</text>
+<text x="16.51" y="-21.59" size="1.778" layer="51" font="vector">Andrew England</text>
 <dimension x1="0" y1="0" x2="38.1" y2="0" x3="19.05" y3="-3.81" textsize="1.778" layer="47" unit="inch"/>
 <dimension x1="0" y1="0" x2="0" y2="25.4" x3="-5.08" y3="12.7" textsize="1.778" layer="47" unit="inch"/>
 <text x="-7.62" y="-36.83" size="1.778" layer="51" font="vector">Black Gloss Soldermask</text>
+<dimension x1="2.54" y1="12.7" x2="2.54" y2="0" x3="-1.27" y3="6.35" textsize="1.778" layer="47" unit="inch"/>
+<dimension x1="2.54" y1="12.7" x2="35.56" y2="12.7" x3="19.05" y3="29.21" textsize="1.778" layer="47" unit="inch"/>
 </plain>
 <attributes>
@@
 <element name="U$11" library="buzzard_labels" package="SCL2" value="" x="32.004" y="22.733" smashed="yes" rot="MR180"/>
 <element name="U$12" library="buzzard_labels" package="SDA1" value="" x="21.844" y="22.733" smashed="yes" rot="MR180"/>
-<element name="U$13" library="buzzard_labels" package="SDA1" value="" x="26.416" y="7.747" smashed="yes" rot="MR0"/>
-<element name="U$14" library="buzzard_labels" package="SCL2" value="" x="36.576" y="7.747" smashed="yes" rot="MR0"/>
+<element name="U$13" library="buzzard_labels" package="SDA1" value="" x="26.543" y="7.747" smashed="yes" rot="MR0"/>
+<element name="U$14" library="buzzard_labels" package="SCL2" value="" x="36.449" y="7.747" smashed="yes" rot="MR0"/>
 <element name="U$15" library="buzzard_labels" package="GND0" value="" x="6.223" y="7.747" smashed="yes" rot="MR0"/>
 <element name="U$16" library="buzzard_labels" package="3V33" value="" x="16.383" y="7.747" smashed="yes" rot="MR0"/>
@@
 <attribute name="VALUE" x="6.477" y="7.366" size="0.6096" layer="27" font="vector" ratio="20" rot="R270" align="top-center"/>
 </element>
-<element name="U$17" library="buzzard_labels (4)" package="GATOR#AIR0" value="" x="26.035" y="12.827" rot="MR0"/>
 <element name="U$19" library="GatorBit_Final_for_Silk#01#png (3)" package="GATORBIT_FINAL_FOR_SILK#01#PNG" value="" x="18.669" y="10.16" rot="MR0"/>
 <element name="R1" library="SparkFun-Resistors" package="0603" value="1k" x="19.05" y="11.43">
 <attribute name="PROD_ID" value="RES-07856" x="19.05" y="11.43" size="1.778" layer="27" display="off"/>
 </element>
-<element name="D4" library="SparkFun-LED" package="LED-0603" value="RED" x="19.05" y="9.525">
-<attribute name="PROD_ID" value="DIO-00819" x="19.05" y="9.525" size="1.778" layer="27" display="off"/>
+<element name="D4" library="SparkFun-LED" package="LED-0603" value="RED" x="19.05" y="7.62">
+<attribute name="PROD_ID" value="DIO-00819" x="19.05" y="7.62" size="1.778" layer="27" display="off"/>
 </element>
 <element name="Q1" library="SparkFun-DiscreteSemi" package="SOT23-3" value="2.5A/30V/105mΩ" x="9.779" y="7.366">
@@
 <attribute name="PROD_ID" value="RES-00824" x="8.89" y="3.81" size="1.778" layer="27" rot="R90" display="off"/>
 </element>
-<element name="U$18" library="buzzard_labels (5)" package="PWR0" value="" x="16.637" y="7.747"/>
+<element name="U$18" library="buzzard_labels (5)" package="PWR0" value="" x="16.637" y="9.525"/>
 <element name="U$20" library="buzzard_labels" package="GND0" value="" x="1.397" y="17.653" smashed="yes" rot="MR180"/>
 <element name="U$21" library="buzzard_labels" package="3V33" value="" x="11.684" y="17.653" smashed="yes" rot="MR180"/>
@@
 <element name="U$23" library="buzzard_labels" package="SCL2" value="" x="32.131" y="17.653" smashed="yes" rot="MR180"/>
 <element name="U$24" library="SparkFun-Aesthetics" package="ORDERING_INSTRUCTIONS" value="" x="-8.89" y="-24.13"/>
+<element name="U$25" library="buzzard_labels (12)" package="GATOR#ENVIRONMENT0" value="" x="32.004" y="12.827" rot="MR0"/>
 </elements>
 <signals>
@@
 <wire x1="17.78" y1="16.295" x2="17.78" y2="15.17" width="0.2032" layer="1"/>
 <contactref element="D1" pad="C"/>
-<wire x1="29.21" y1="4.96" x2="29.21" y2="7.62" width="0.2032" layer="1"/>
-<wire x1="29.21" y1="7.62" x2="32.385" y2="10.795" width="0.2032" layer="1"/>
 <contactref element="J1" pad="P$2"/>
-<wire x1="34.29" y1="3.556" x2="34.29" y2="8.89" width="0.2032" layer="1"/>
+<wire x1="34.29" y1="3.556" x2="34.29" y2="5.08" width="0.2032" layer="1"/>
+<wire x1="34.29" y1="5.08" x2="34.29" y2="8.89" width="0.2032" layer="1"/>
+<wire x1="29.21" y1="4.96" x2="29.33" y2="5.08" width="0.2032" layer="1"/>
+<wire x1="29.33" y1="5.08" x2="34.29" y2="5.08" width="0.2032" layer="1"/>
 </signal>
 <signal name="SDA">
@@
 <wire x1="24.257" y1="14.295" x2="26.915" y2="14.295" width="0.2032" layer="1"/>
 <contactref element="D2" pad="C"/>
-<wire x1="19.05" y1="4.96" x2="19.05" y2="6.35" width="0.2032" layer="1"/>
-<wire x1="19.05" y1="6.35" x2="21.59" y2="8.89" width="0.2032" layer="1"/>
-<wire x1="21.59" y1="8.89" x2="24.13" y2="8.89" width="0.2032" layer="1"/>
 <wire x1="22.098" y1="16.256" x2="22.479" y2="15.875" width="0.2032" layer="16"/>
 <contactref element="J2" pad="P$2"/>
 <wire x1="24.13" y1="3.556" x2="24.13" y2="8.89" width="0.2032" layer="1"/>
+<wire x1="24.13" y1="3.556" x2="22.726" y2="4.96" width="0.2032" layer="1"/>
+<wire x1="22.726" y1="4.96" x2="19.05" y2="4.96" width="0.2032" layer="1"/>
 </signal>
 <signal name="3.3V">
@@
 <contactref element="R1" pad="1"/>
 <wire x1="18.2" y1="11.43" x2="18.173" y2="11.403" width="0.2032" layer="1"/>
-<wire x1="18.173" y1="11.403" x2="18.173" y2="9.525" width="0.2032" layer="1"/>
+<wire x1="18.173" y1="11.403" x2="18.173" y2="7.62" width="0.2032" layer="1"/>
 </signal>
 <signal name="N$3">
@@
 <wire x1="10.16" y1="3.81" x2="9.779" y2="4.191" width="0.2032" layer="1"/>
 <wire x1="9.779" y1="4.191" x2="9.779" y2="8.466" width="0.2032" layer="1"/>
-<wire x1="13.97" y1="21.844" x2="13.97" y2="12.446" width="0.2032" layer="16"/>
-<via x="13.97" y="12.446" extent="1-16" drill="0.381"/>
-<wire x1="13.97" y1="12.446" x2="13.97" y2="3.81" width="0.2032" layer="1"/>
+<wire x1="13.97" y1="21.844" x2="13.97" y2="8.89" width="0.3048" layer="16"/>
+<via x="13.97" y="8.89" extent="1-16" drill="0.381"/>
+<wire x1="13.97" y1="8.89" x2="13.97" y2="3.81" width="0.3048" layer="1"/>
 <wire x1="13.97" y1="3.81" x2="13.843" y2="3.683" width="0.2032" layer="1"/>
 </signal>

Commit message: updating pwrsilk
Parts:
- U$18: device buzzard_labels (5):PWR0 -> buzzard_labels (13):PWR0
- moved D4 1.91 mm to (19.1, 9.53)
- moved U$18 1.78 mm to (16.6, 7.75)
Routing:
- net N$2: track 3.82 -> 1.92 mm
Changed lines of the file:
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@@
 <attribute name="PROD_ID" value="RES-07856" x="19.05" y="11.43" size="1.778" layer="27" display="off"/>
 </element>
-<element name="D4" library="SparkFun-LED" package="LED-0603" value="RED" x="19.05" y="7.62">
-<attribute name="PROD_ID" value="DIO-00819" x="19.05" y="7.62" size="1.778" layer="27" display="off"/>
+<element name="D4" library="SparkFun-LED" package="LED-0603" value="RED" x="19.05" y="9.525">
+<attribute name="PROD_ID" value="DIO-00819" x="19.05" y="9.525" size="1.778" layer="27" display="off"/>
 </element>
 <element name="Q1" library="SparkFun-DiscreteSemi" package="SOT23-3" value="2.5A/30V/105mΩ" x="9.779" y="7.366">
@@
 <attribute name="PROD_ID" value="RES-00824" x="8.89" y="3.81" size="1.778" layer="27" rot="R90" display="off"/>
 </element>
-<element name="U$18" library="buzzard_labels (5)" package="PWR0" value="" x="16.637" y="9.525"/>
+<element name="U$18" library="buzzard_labels (13)" package="PWR0" value="" x="16.637" y="7.747"/>
 <element name="U$20" library="buzzard_labels" package="GND0" value="" x="1.397" y="17.653" smashed="yes" rot="MR180"/>
 <element name="U$21" library="buzzard_labels" package="3V33" value="" x="11.684" y="17.653" smashed="yes" rot="MR180"/>
@@
 <contactref element="R1" pad="1"/>
 <wire x1="18.2" y1="11.43" x2="18.173" y2="11.403" width="0.2032" layer="1"/>
-<wire x1="18.173" y1="11.403" x2="18.173" y2="7.62" width="0.2032" layer="1"/>
+<wire x1="18.173" y1="11.403" x2="18.173" y2="9.525" width="0.2032" layer="1"/>
 </signal>
 <signal name="N$3">

Commit message: QC Double check changes
Parts:
- removed U$10: (no value), buzzard_labels:GND0
- removed U$11: (no value), buzzard_labels:SCL2
- removed U$12: (no value), buzzard_labels:SDA1
- removed U$9: (no value), buzzard_labels:3V33
Changed lines of the file:
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@@
 <element name="U$7" library="buzzard_labels" package="GND0" value="" x="6.223" y="17.653" smashed="yes" rot="R180"/>
 <element name="U$8" library="buzzard_labels" package="3V33" value="" x="16.383" y="17.653" smashed="yes" rot="R180"/>
-<element name="U$9" library="buzzard_labels" package="3V33" value="" x="11.684" y="22.733" smashed="yes" rot="MR180"/>
-<element name="U$10" library="buzzard_labels" package="GND0" value="" x="1.397" y="22.733" smashed="yes" rot="MR180"/>
-<element name="U$11" library="buzzard_labels" package="SCL2" value="" x="32.004" y="22.733" smashed="yes" rot="MR180"/>
-<element name="U$12" library="buzzard_labels" package="SDA1" value="" x="21.844" y="22.733" smashed="yes" rot="MR180"/>
 <element name="U$13" library="buzzard_labels" package="SDA1" value="" x="26.543" y="7.747" smashed="yes" rot="MR0"/>
 <element name="U$14" library="buzzard_labels" package="SCL2" value="" x="36.449" y="7.747" smashed="yes" rot="MR0"/>
@@
 <contactref element="R5" pad="1"/>
 <via x="15.24" y="8.89" extent="1-16" drill="0.381"/>
+<via x="15.875" y="16.383" extent="1-16" drill="0.381"/>
+<via x="22.86" y="8.89" extent="1-16" drill="0.381"/>
+<via x="25.4" y="8.89" extent="1-16" drill="0.381"/>
 </signal>
 <signal name="SCL">
